File: pcb/USB2BLE.kicad_pcb (KiCad board)
At the start: 2 copper layers, 27.6 x 33 mm, 11 parts, among them J1 Conn_01x02, SW1 SW_SPDT, U1 XIAO-ESP32-S3-SMD, U2 MT3608

Commit message: updated
Parts:
- added C3: 30p, Capacitor_SMD:C_0805_2012Metric_Pad1.18x1.45mm_HandSolder, F.Cu at (131.0, 85.5)
- C1, C2: value C -> 22uF
- L1: value L -> 22uH
- moved U2 10.3 mm to (121.0, 87.0), turned to 0 degrees
- moved C2 8.76 mm to (134.0, 87.5), turned to 90 degrees
- moved L1 7.60 mm to (124.5, 88.0), turned to -90 degrees
- moved D1 6.77 mm to (129.4, 88.5)
- moved C1 6.66 mm to (121.2, 89.8), turned to 180 degrees
- moved SW1 4.51 mm to (122.4, 93.0)
- moved R2 4.12 mm to (131.0, 81.5)
- moved R1 1.36 mm to (131.0, 83.5)
Connections:
- C1 pad 1: GND -> /VBAT
- C1 pad 2: /VBAT -> GND
- U1 pad 14: unconnected-(U1-VBUS-Pad14) -> /5V_OUT
Routing:
- net /5V_OUT: track 17.2 -> 33.3 mm
- net Net-(U2-FB): track 7.17 -> 19.9 mm
- net Net-(D1-K): track 17.5 -> 12.7 mm
- net Net-(J1-Pin_1): track 10.5 -> 15.2 mm
- net /VBAT: track 36.0 -> 32.5 mm
- net GND: track 16.6 -> 18.2 mm, vias 3 -> 5
